File: PCB Template/PCB Template.kicad_sch (KiCad schematic)
At the start: 8 parts, among them J1 ESL_PQ_MainHeader, J2 Conn_01x04, U1 STM32L476RGTx, U2 MAX485ESA+T

Commit message: Niel 1
Other:
- added sheet Chris (untitled.kicad_sch)
Changed lines of the file:
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@@
+		)
+	)
+	(sheet
+		(at 229.87 137.16)
+		(size 43.18 21.59)
+		(fields_autoplaced yes)
+		(stroke
+			(width 0.1524)
+			(type solid)
+		)
+		(fill
+			(color 0 0 0 0.0000)
+		)
+		(property "Sheetname" "Chris"
+			(at 229.87 136.4484 0)
+			(effects
+				(font
+					(size 1.27 1.27)
+				)
+				(justify left bottom)
+			)
+		)
+		(property "Sheetfile" "untitled.kicad_sch"
+			(at 229.87 159.3346 0)
+			(effects
+				(font
+					(size 1.27 1.27)
+				)
+				(justify left top)
+			)
+		)
+		(pin "Output" input
+			(at 273.05 147.32 0)
+			(effects
+				(font
+					(size 1.27 1.27)
+				)
+				(justify right)
+			)
+		)
+		(instances
+			(project "PCB Template"
+				(path "/2108ba15-8357-4ea6-b863-64720f006d55"
+					(page "2")
+				)
+			)
 		)
 	)
